File: hardware/reflowoven.sch (KiCad schematic (older format))
At the start: 25 parts, among them P1 USB-A-SHLD, P2 CONN_6, P3 CONN_2, P5 CONN_2, U1 FT232RL, U2 255-3100-ND, U3 MSP430G2553IPW20, U4 AD594/95, U5 LM317, X1 CRYSTAL

Commit message: First round of changes to add additional relays and thermal couples
Parts:
- removed D1: DIODE, D4, symbol DIODE
- removed U2: 255-3100-ND, symbol 255-3100-ND
- removed U4: AD594/95, DIP-14__300, symbol AD594/95
- added DA1, DA2: AD8495, Housings_SSOP:MSOP-8_3x3mm_Pitch0.65mm, symbol AD8495
- added P5: CONN_01X08, svolpe-custom-mod:1935226, symbol CONN_01X08
- added U4, U6, U7, U8: MCHRM3H, svolpe-custom-mod:MCHRM3H, symbol MCHRM3H
- added U5: ULN2003A, symbol ULN2003A
- C1: renamed from C7; footprint (none) -> Capacitors_SMD:C_0603; symbol C -> C-RESCUE-reflowoven
- C2: renamed from C1; footprint (none) -> Capacitors_SMD:C_0603; symbol C -> C-RESCUE-reflowoven
- C3: renamed from C2; footprint (none) -> Capacitors_SMD:C_0603; symbol C -> C-RESCUE-reflowoven
- C4: renamed from C3; footprint (none) -> Capacitors_SMD:C_0603; symbol C -> C-RESCUE-reflowoven
- C5: renamed from C4; footprint (none) -> Capacitors_SMD:C_0805; symbol CP1 -> C
- C6: renamed from C5; footprint (none) -> Capacitors_SMD:C_0603; symbol C -> C-RESCUE-reflowoven
- D1: renamed from D2; footprint (none) -> LEDs:LED_D4.0mm; symbol LED -> LED-RESCUE-reflowoven
- D2: renamed from D3; footprint (none) -> LEDs:LED_D4.0mm; symbol LED -> LED-RESCUE-reflowoven
- P1: footprint (none) -> Connectors:USB_B
- P3: footprint (none) -> svolpe-custom-mod:1751248
- P4: renamed from P5; footprint (none) -> svolpe-custom-mod:1751248
- R1: renamed from R4; footprint (none) -> Resistors_SMD:R_1206
- R2, R3: footprint (none) -> Resistors_SMD:R_0603
- R4: renamed from R1; footprint (none) -> Resistors_SMD:R_0603
- R5, R6: footprint (none) -> Resistors_SMD:R_0603; symbol R -> R-RESCUE-reflowoven
- U1: footprint SSOP28 -> Housings_SSOP:SSOP-28_5.3x10.2mm_Pitch0.65mm
- U2: renamed from U3; footprint (none) -> Housings_SSOP:TSSOP-20_4.4x6.5mm_Pitch0.65mm
- U3: renamed from U5; footprint (none) -> TO_SOT_Packages_THT:TO-220_Vertical
- X1: footprint (none) -> Crystals:Crystal_Round_d1.0mm_Vertical
Connections:
- net labels added: THERMOCOUPLE_1+, THERMOCOUPLE_1-, THERMOCOUPLE_2+, THERMOCOUPLE_2-
- net labels removed: THERMOCOUPLE-
- wire segments 87 -> 101
- no-connect marks 32 -> 28
Other:
- moved on the sheet: P3, P4

Commit message: Finalized layout with 2 thermocouples and 4 relays
Parts:
- removed DA1, DA2: AD8495, Housings_SSOP:MSOP-8_3x3mm_Pitch0.65mm, symbol AD8495
- removed U1: FT232RL, Housings_SSOP:SSOP-28_5.3x10.2mm_Pitch0.65mm, symbol FT232RL
- removed U4, U6, U7, U8: MCHRM3H, svolpe-custom-mod:MCHRM3H, symbol MCHRM3H
- removed U5: ULN2003A, symbol ULN2003A
- added U2: FT232RL, Housings_SSOP:SSOP-28_5.3x10.2mm_Pitch0.65mm, symbol FT232RL
- P2: footprint (none) -> Pin_Headers:Pin_Header_Straight_1x06_Pitch2.54mm
- renumbered U2 to U1
Connections:
- net labels added: +5V, TEMP_1, TEMP_2
- net labels removed: TEMP, THERMOCOUPLE+, THERMOCOUPLE_1+, THERMOCOUPLE_1-, THERMOCOUPLE_2+, THERMOCOUPLE_2-
- wire segments 101 -> 125
- no-connect marks 28 -> 17
Other:
- moved on the sheet: C5, P2, R2, R3, R4, U1, X1

Commit message: cleaned up schematic some
Connections:
- wire segments 125 -> 110
Changed lines of the file:
@@
 	2050 5100 1800 5100
 Wire Wire Line
-	1800 5300 2450 5300
-Wire Wire Line
-	2450 5300 3300 5300
+	1800 5300 3300 5300
 Wire Wire Line
 	1800 5400 2050 5400
@@
 	2350 5200 1800 5200
 Wire Wire Line
-	2450 5150 2450 5300
-Wire Wire Line
-	2450 5300 2450 5450
+	2450 5150 2450 5450
 Connection ~ 2450 5300
 Wire Wire Line
 	2450 4750 2050 4750
 Wire Wire Line
-	2050 5850 2200 5850
-Wire Wire Line
-	2200 5850 2450 5850
+	2050 5850 2450 5850
 Wire Wire Line
 	2200 5900 2200 5850
@@
 	3550 6450 3550 6350
 Wire Wire Line
-	3550 6850 3850 6850
-Wire Wire Line
-	3850 6850 4150 6850
+	3550 6850 4150 6850
 Wire Wire Line
 	3850 6950 3850 6850
@@
 	1250 4000 1100 4000
 Wire Wire Line
-	1100 4000 1100 4450
-Wire Wire Line
-	1100 4450 1100 4600
+	1100 4000 1100 4600
 Wire Wire Line
 	1100 4450 1250 4450
@@
 	3300 5700 3050 5700
 Wire Wire Line
-	4900 3450 4900 3550
+	4900 3450 4900 3800
 Wire Wire Line
-	4900 3550 4900 3800
-Wire Wire Line
-	4900 3550 5300 3550
-Wire Wire Line
-	5300 3550 5650 3550
+	4900 3550 5650 3550
 Connection ~ 4900 3550
 Connection ~ 5300 3550
 Wire Wire Line
-	5300 3950 5500 3950
-Wire Wire Line
-	5500 3950 5650 3950
+	5300 3950 5650 3950
 Wire Wire Line
 	5500 4000 5500 3950
@@
 	2450 4750 2450 4850
 Wire Wire Line
-	2850 1400 2100 1400
-Wire Wire Line
-	2100 1400 1950 1400
+	1950 1400 2850 1400
 Wire Wire Line
 	2200 1800 1950 1800
@@
 	2200 1600 1950 1600
 Wire Wire Line
-	1950 2000 1950 2400
-Wire Wire Line
-	1950 2400 1950 2500
+	1950 2000 1950 2500
 Wire Wire Line
 	1800 2400 1950 2400
@@
 	3800 3250 3800 3350
 Wire Wire Line
-	6200 950  6450 950
-Wire Wire Line
-	6450 950  6850 950
+	6200 950  6850 950
 Wire Wire Line
 	6850 950  6850 900
@@
 	6600 2050 6450 2050
 Wire Wire Line
-	6450 1450 6450 1500
-Wire Wire Line
-	6450 1500 6450 1550
+	6450 1450 6450 1550
 Wire Wire Line
 	6450 1500 5800 1500
@@
 	6600 2200 6600 2050
 Wire Wire Line
-	3500 3250 3650 3250
-Wire Wire Line
-	3650 3250 3800 3250
-Wire Wire Line
-	3800 3250 3950 3250
-Wire Wire Line
-	3950 3250 4100 3250
+	3500 3250 4100 3250
 Connection ~ 3650 3250
 Connection ~ 3950 3250

Commit message: Update schematic to reflect proper resistor values for 3.3V regulator
Parts:
- R5: value 330 -> 750
- R6: value 560 -> 2K
Other:
- note added: "R5 + 1"
- note added: "R6"
- note added: "Vo = 1.25V x"
Changed lines of the file:
@@
 P 6450 1200
 F 0 "R5" V 6530 1200 50  0000 C CNN
-F 1 "330" V 6450 1200 50  0000 C CNN
+F 1 "750" V 6450 1200 50  0000 C CNN
 F 2 "Resistors_SMD:R_0603" H 6450 1200 60  0001 C CNN
 F 3 "" H 6450 1200 60  0001 C CNN
@@
 P 6450 1800
 F 0 "R6" V 6530 1800 50  0000 C CNN
-F 1 "560" V 6450 1800 50  0000 C CNN
+F 1 "2K" V 6450 1800 50  0000 C CNN
 F 2 "Resistors_SMD:R_0603" H 6450 1800 60  0001 C CNN
 F 3 "" H 6450 1800 60  0001 C CNN
@@
 	1    0    0    -1
 $EndComp
+Text Notes 7680 930  0    60   ~ 0
+R6
+Text Notes 7580 1030 0    60   ~ 0
+R5 + 1
+Wire Notes Line
+	7580 930  7880 930
+Text Notes 6930 960  0    60   ~ 0
+Vo = 1.25V x
 $EndSCHEMATC
