File: hardware/reflowoven.sch (KiCad schematic (older format))
At the start: 23 parts, among them P1 USB-A-SHLD, P2 CONN_6, P3 CONN_2, P4 CONN_2, P5 CONN_01X08, U1 MSP430G2553IPW20, U2 FT232RL, U3 LM317, X1 CRYSTAL

Commit message: Change thermocouple circuitry from 5V to 3.3V
Changed lines of the file:
@@
 $EndComp
 $Comp
-L +3.3V-RESCUE-reflowoven #PWR01
-U 1 1 50F87C90
-P 4900 3450
-F 0 "#PWR01" H 4900 3410 30  0001 C CNN
-F 1 "+3.3V" H 4900 3560 30  0000 C CNN
-F 2 "" H 4900 3450 60  0001 C CNN
-F 3 "" H 4900 3450 60  0001 C CNN
-	1    4900 3450
-	1    0    0    -1
-$EndComp
-$Comp
-L GND-RESCUE-reflowoven #PWR02
+L GND-RESCUE-reflowoven #PWR01
 U 1 1 50F87C99
 P 4900 6150
-F 0 "#PWR02" H 4900 6150 30  0001 C CNN
+F 0 "#PWR01" H 4900 6150 30  0001 C CNN
 F 1 "GND" H 4900 6080 30  0001 C CNN
 F 2 "" H 4900 6150 60  0001 C CNN
 F 3 "" H 4900 6150 60  0001 C CNN
 	1    4900 6150
-	1    0    0    -1
-$EndComp
-$Comp
-L +3.3V-RESCUE-reflowoven #PWR03
-U 1 1 50F8B4DA
-P 2050 4750
-F 0 "#PWR03" H 2050 4710 30  0001 C CNN
-F 1 "+3.3V" H 2050 4860 30  0000 C CNN
-F 2 "" H 2050 4750 60  0001 C CNN
-F 3 "" H 2050 4750 60  0001 C CNN
-	1    2050 4750
 	1    0    0    -1
 $EndComp
@@
 $EndComp
 $Comp
-L GND-RESCUE-reflowoven #PWR04
+L GND-RESCUE-reflowoven #PWR02
 U 1 1 50FB89AB
 P 2200 5900
-F 0 "#PWR04" H 2200 5900 30  0001 C CNN
+F 0 "#PWR02" H 2200 5900 30  0001 C CNN
 F 1 "GND" H 2200 5830 30  0001 C CNN
 F 2 "" H 2200 5900 60  0001 C CNN
@@
 $EndComp
 $Comp
-L GND-RESCUE-reflowoven #PWR05
+L GND-RESCUE-reflowoven #PWR03
 U 1 1 50FB94DA
 P 3850 6950
-F 0 "#PWR05" H 3850 6950 30  0001 C CNN
+F 0 "#PWR03" H 3850 6950 30  0001 C CNN
 F 1 "GND" H 3850 6880 30  0001 C CNN
 F 2 "" H 3850 6950 60  0001 C CNN
@@
 $EndComp
 $Comp
-L GND-RESCUE-reflowoven #PWR06
+L GND-RESCUE-reflowoven #PWR04
 U 1 1 50FC20B8
 P 1100 4600
-F 0 "#PWR06" H 1100 4600 30  0001 C CNN
+F 0 "#PWR04" H 1100 4600 30  0001 C CNN
 F 1 "GND" H 1100 4530 30  0001 C CNN
 F 2 "" H 1100 4600 60  0001 C CNN
@@
 $EndComp
 $Comp
-L GND-RESCUE-reflowoven #PWR07
+L GND-RESCUE-reflowoven #PWR05
 U 1 1 51008987
 P 5500 4000
-F 0 "#PWR07" H 5500 4000 30  0001 C CNN
+F 0 "#PWR05" H 5500 4000 30  0001 C CNN
 F 1 "GND" H 5500 3930 30  0001 C CNN
 F 2 "" H 5500 4000 60  0001 C CNN
@@
 $EndComp
 $Comp
-L GND-RESCUE-reflowoven #PWR08
+L GND-RESCUE-reflowoven #PWR06
 U 1 1 58BC3A9D
 P 1950 2500
-F 0 "#PWR08" H 1950 2500 30  0001 C CNN
+F 0 "#PWR06" H 1950 2500 30  0001 C CNN
 F 1 "GND" H 1950 2430 30  0001 C CNN
 F 2 "" H 1950 2500 60  0001 C CNN
@@
 $EndComp
 $Comp
-L GND-RESCUE-reflowoven #PWR09
+L GND-RESCUE-reflowoven #PWR07
 U 1 1 58BD0915
 P 3800 3350
-F 0 "#PWR09" H 3800 3350 30  0001 C CNN
+F 0 "#PWR07" H 3800 3350 30  0001 C CNN
 F 1 "GND" H 3800 3280 30  0001 C CNN
 F 2 "" H 3800 3350 60  0001 C CNN
 F 3 "" H 3800 3350 60  0001 C CNN
 	1    3800 3350
-	1    0    0    -1
-$EndComp
-$Comp
-L +3.3V-RESCUE-reflowoven #PWR010
-U 1 1 58BD091B
-P 6850 900
-F 0 "#PWR010" H 6850 860 30  0001 C CNN
-F 1 "+3.3V" H 6850 1010 30  0000 C CNN
-F 2 "" H 6850 900 60  0001 C CNN
-F 3 "" H 6850 900 60  0001 C CNN
-	1    6850 900
 	1    0    0    -1
 $EndComp
@@
 VBUS
 $Comp
-L GND-RESCUE-reflowoven #PWR011
+L GND-RESCUE-reflowoven #PWR08
 U 1 1 58BD0926
 P 6600 2200
-F 0 "#PWR011" H 6600 2200 30  0001 C CNN
+F 0 "#PWR08" H 6600 2200 30  0001 C CNN
 F 1 "GND" H 6600 2130 30  0001 C CNN
 F 2 "" H 6600 2200 60  0001 C CNN
@@
 NoConn ~ 2850 2250
 NoConn ~ 2850 2050
-$Comp
-L +3.3V-RESCUE-reflowoven #PWR012
-U 1 1 58BD095D
-P 2800 1150
-F 0 "#PWR012" H 2800 1110 30  0001 C CNN
-F 1 "+3.3V" H 2800 1260 30  0000 C CNN
-F 2 "" H 2800 1150 60  0001 C CNN
-F 3 "" H 2800 1150 60  0001 C CNN
-	1    2800 1150
-	1    0    0    -1
-$EndComp
 Text Label 6550 3050 0    60   ~ 0
 TEMP_1
@@
 TEMP_2
 $Comp
-L +5V #PWR013
+L +5V #PWR09
 U 1 1 58BE4EB3
 P 2100 1050
-F 0 "#PWR013" H 50  -50 50  0001 C CNN
+F 0 "#PWR09" H 50  -50 50  0001 C CNN
 F 1 "+5V" H 2115 1223 50  0000 C CNN
 F 2 "" H 50  100 50  0001 C CNN
@@
 $EndComp
 $Comp
-L +5V #PWR014
+L +5V #PWR010
 U 1 1 58BE558A
 P 6250 3450
-F 0 "#PWR014" H 0   0   50  0001 C CNN
+F 0 "#PWR010" H 0   0   50  0001 C CNN
 F 1 "+5V" H 6265 3623 50  0000 C CNN
 F 2 "" H 0   150 50  0001 C CNN
@@
 	2650 2550 2650 2600
 $Comp
-L GND #PWR015
+L GND #PWR011
 U 1 1 58BE58A9
 P 2650 3000
-F 0 "#PWR015" H 0   -350 50  0001 C CNN
+F 0 "#PWR011" H 0   -350 50  0001 C CNN
 F 1 "GND" H 2655 2827 50  0000 C CNN
 F 2 "" H 0   -100 50  0001 C CNN
@@
 Text Notes 6930 960  0    60   ~ 0
 Vo = 1.25V x
+$Comp
+L +3.3V #PWR012
+U 1 1 58D854D1
+P 2800 1150
+F 0 "#PWR012" H -150 200 50  0001 C CNN
+F 1 "+3.3V" H 2815 1323 50  0000 C CNN
+F 2 "" H -150 350 50  0001 C CNN
+F 3 "" H -150 350 50  0001 C CNN
+	1    2800 1150
+	1    0    0    -1
+$EndComp
+$Comp
+L +3.3V #PWR013
+U 1 1 58D85715
+P 6850 900
+F 0 "#PWR013" H 0   -50 50  0001 C CNN
+F 1 "+3.3V" H 6865 1073 50  0000 C CNN
+F 2 "" H 0   100 50  0001 C CNN
+F 3 "" H 0   100 50  0001 C CNN
+	1    6850 900
+	1    0    0    -1
+$EndComp
+$Comp
+L +3.3V #PWR014
+U 1 1 58D86E74
+P 2050 4750
+F 0 "#PWR014" H -550 350 50  0001 C CNN
+F 1 "+3.3V" H 2065 4923 50  0000 C CNN
+F 2 "" H -550 500 50  0001 C CNN
+F 3 "" H -550 500 50  0001 C CNN
+	1    2050 4750
+	1    0    0    -1
+$EndComp
+$Comp
+L +3.3V #PWR015
+U 1 1 58D86F28
+P 4900 3450
+F 0 "#PWR015" H -50 -150 50  0001 C CNN
+F 1 "+3.3V" H 4915 3623 50  0000 C CNN
+F 2 "" H -50 0   50  0001 C CNN
+F 3 "" H -50 0   50  0001 C CNN
+	1    4900 3450
+	1    0    0    -1
+$EndComp
 $EndSCHEMATC

Commit message: Update schematic and PCB to include additional 1M ohm resitor on thermocouple - term.  This seems to stablize the temp readings.
Parts:
- C5: symbol C -> C-RESCUE-reflowoven
- D1, D2: symbol LED-RESCUE-reflowoven -> LED
- R1, R2, R3, R4: symbol R -> R-RESCUE-reflowoven
Connections:
- wire segments 109 -> 106
Changed lines of the file:
@@
 LIBS:analog_devices
 LIBS:svolpe-custom
+LIBS:diode
 LIBS:reflowoven-cache
 EELAYER 26 0
@@
 $EndComp
 $Comp
-L R R4
+L R-RESCUE-reflowoven R4
 U 1 1 50FB89E1
 P 2450 5000
@@
 TCK
 $Comp
-L LED-RESCUE-reflowoven D1
+L LED D1
 U 1 1 50FC1D40
-P 1450 4000
-F 0 "D1" H 1450 4100 50  0000 C CNN
-F 1 "LED" H 1450 3900 50  0000 C CNN
-F 2 "LEDs:LED_D4.0mm" H 1450 4000 60  0001 C CNN
-F 3 "" H 1450 4000 60  0001 C CNN
-	1    1450 4000
-	-1   0    0    1
-$EndComp
-$Comp
-L LED-RESCUE-reflowoven D2
+P 1500 4000
+F 0 "D1" H 1500 4100 50  0000 C CNN
+F 1 "LED" H 1500 3900 50  0000 C CNN
+F 2 "LEDs:LED_D4.0mm" H 1500 4000 60  0001 C CNN
+F 3 "" H 1500 4000 60  0001 C CNN
+	1    1500 4000
+	1    0    0    -1
+$EndComp
+$Comp
+L LED D2
 U 1 1 50FC1D4F
-P 1450 4450
-F 0 "D2" H 1450 4550 50  0000 C CNN
-F 1 "LED" H 1450 4350 50  0000 C CNN
-F 2 "LEDs:LED_D4.0mm" H 1450 4450 60  0001 C CNN
-F 3 "" H 1450 4450 60  0001 C CNN
-	1    1450 4450
-	-1   0    0    1
-$EndComp
-$Comp
-L R R2
+P 1500 4450
+F 0 "D2" H 1500 4550 50  0000 C CNN
+F 1 "LED" H 1500 4350 50  0000 C CNN
+F 2 "LEDs:LED_D4.0mm" H 1500 4450 60  0001 C CNN
+F 3 "" H 1500 4450 60  0001 C CNN
+	1    1500 4450
+	1    0    0    -1
+$EndComp
+$Comp
+L R-RESCUE-reflowoven R2
 U 1 1 50FC1D77
 P 2050 4000
@@
 $EndComp
 $Comp
-L R R3
+L R-RESCUE-reflowoven R3
 U 1 1 50FC1D9D
 P 2050 4450
@@
 $EndComp
 $Comp
-L C C5
+L C-RESCUE-reflowoven C5
 U 1 1 51008DD5
 P 5300 3750
@@
 $EndComp
 $Comp
-L R R1
+L R-RESCUE-reflowoven R1
 U 1 1 58BC3AA3
 P 1650 2400
@@
 Wire Wire Line
 	2350 5200 1800 5200
-Wire Wire Line
-	2450 5150 2450 5450
 Connection ~ 2450 5300
-Wire Wire Line
-	2450 4750 2050 4750
 Wire Wire Line
 	2050 5850 2450 5850
@@
 Connection ~ 3850 6850
 Wire Wire Line
-	1650 4000 1900 4000
-Wire Wire Line
-	1650 4450 1900 4450
-Wire Wire Line
-	1250 4000 1100 4000
+	1350 4000 1100 4000
 Wire Wire Line
 	1100 4000 1100 4600
 Wire Wire Line
-	1100 4450 1250 4450
+	1100 4450 1350 4450
 Connection ~ 1100 4450
-Wire Wire Line
-	2200 4000 3200 4000
 Wire Wire Line
 	3300 5600 3050 5600
@@
 Connection ~ 5300 3550
 Wire Wire Line
-	5300 3950 5650 3950
-Wire Wire Line
 	5500 4000 5500 3950
 Connection ~ 5500 3950
 Wire Wire Line
-	2200 4450 2700 4450
-Wire Wire Line
 	3300 4400 3200 4400
 Wire Wire Line
@@
 	2700 5000 3300 5000
 Wire Wire Line
-	2450 4750 2450 4850
-Wire Wire Line
 	1950 1400 2850 1400
 Wire Wire Line
@@
 Wire Wire Line
 	1950 2000 1950 2500
-Wire Wire Line
-	1800 2400 1950 2400
 Connection ~ 1950 2400
-Wire Wire Line
-	1350 2400 1500 2400
 Wire Wire Line
 	1350 2400 1350 2350
@@
 	6950 3200 6550 3200
 Wire Wire Line
-	5300 3600 5300 3550
-Wire Wire Line
-	5300 3900 5300 3950
-Wire Wire Line
 	6400 3750 6950 3750
 Wire Wire Line
@@
 	2650 2550 2650 2600
 $Comp
-L GND #PWR011
+L GND-RESCUE-reflowoven #PWR011
 U 1 1 58BE58A9
 P 2650 3000
@@
 Vo = 1.25V x
 $Comp
-L +3.3V #PWR012
+L +3.3V-RESCUE-reflowoven #PWR012
 U 1 1 58D854D1
 P 2800 1150
@@
 $EndComp
 $Comp
-L +3.3V #PWR013
+L +3.3V-RESCUE-reflowoven #PWR013
 U 1 1 58D85715
 P 6850 900
@@
 $EndComp
 $Comp
-L +3.3V #PWR014
+L +3.3V-RESCUE-reflowoven #PWR014
 U 1 1 58D86E74
 P 2050 4750
 F 0 "#PWR014" H -550 350 50  0001 C CNN
-F 1 "+3.3V" H 2065 4923 50  0000 C CNN
+F 1 "+3.3V" H 2200 4850 50  0000 C CNN
 F 2 "" H -550 500 50  0001 C CNN
 F 3 "" H -550 500 50  0001 C CNN
@@
 $EndComp
 $Comp
-L +3.3V #PWR015
+L +3.3V-RESCUE-reflowoven #PWR015
 U 1 1 58D86F28
 P 4900 3450
@@
 	1    0    0    -1
 $EndComp
+Wire Wire Line
+	1800 4000 1650 4000
+Wire Wire Line
+	1800 4450 1650 4450
+Wire Wire Line
+	2300 4450 2700 4450
+Wire Wire Line
+	3200 4000 2300 4000
+Wire Wire Line
+	2450 4750 2050 4750
+Wire Wire Line
+	2450 5250 2450 5450
+Wire Wire Line
+	5300 3950 5650 3950
+Wire Wire Line
+	1350 2400 1400 2400
+Wire Wire Line
+	1900 2400 1950 2400
 $EndSCHEMATC
