File: hardware/Relays and Themocouples.sch (KiCad schematic (older format))
At the start: 17 parts, among them U4 ULN2003A, U5 MCHRM3H, U6 MCHRM3H, U7 MCHRM3H, U8 MCHRM3H

Commit message: Update PCB to change thermocouples to 3.3V.  Update command interface to convert temp to degrees instead of sending raw ADC
Connections:
- net labels added: +3.3V
- net labels removed: +5V
Other:
- note added: "5mV/C"
- note added: "Red wire"
- note added: "Yellow wire"
Changed lines of the file:
@@
 Wire Wire Line
 	5500 1400 5500 1000
-$Comp
-L +5V #PWR021
-U 1 1 58BCE305
-P 5500 1000
-F 0 "#PWR021" H -50 -50 50  0001 C CNN
-F 1 "+5V" H 5515 1173 50  0000 C CNN
-F 2 "" H -50 100 50  0001 C CNN
-F 3 "" H -50 100 50  0001 C CNN
-	1    5500 1000
-	1    0    0    -1
-$EndComp
-$Comp
-L +5V #PWR022
-U 1 1 58BCE39A
-P 5500 2200
-F 0 "#PWR022" H -150 50  50  0001 C CNN
-F 1 "+5V" H 5515 2373 50  0000 C CNN
-F 2 "" H -150 200 50  0001 C CNN
-F 3 "" H -150 200 50  0001 C CNN
-	1    5500 2200
-	1    0    0    -1
-$EndComp
 Wire Wire Line
 	6050 2650 6050 2400
@@
 Wire Wire Line
 	7250 1900 7250 2350
+Text Notes 10100 1500 0    60   ~ 0
+Yellow wire
+Text Notes 10100 1250 0    60   ~ 0
+Red wire
+Text Notes 3800 1100 0    60   ~ 0
+5mV/C
+$Comp
+L +3.3V #PWR021
+U 1 1 58D7F88C
+P 5500 1000
+F 0 "#PWR021" H 1300 0   50  0001 C CNN
+F 1 "+3.3V" H 5515 1173 50  0000 C CNN
+F 2 "" H 1300 150 50  0001 C CNN
+F 3 "" H 1300 150 50  0001 C CNN
+	1    5500 1000
+	1    0    0    -1
+$EndComp
+$Comp
+L +3.3V #PWR022
+U 1 1 58D7FA01
+P 5500 2200
+F 0 "#PWR022" H 1300 1200 50  0001 C CNN
+F 1 "+3.3V" H 5515 2373 50  0000 C CNN
+F 2 "" H 1300 1350 50  0001 C CNN
+F 3 "" H 1300 1350 50  0001 C CNN
+	1    5500 2200
+	1    0    0    -1
+$EndComp
 $EndSCHEMATC

Commit message: Update schematic and PCB to include additional 1M ohm resitor on thermocouple - term.  This seems to stablize the temp readings.
Parts:
- added R11, R12: 1M, Resistors_SMD:R_0603, symbol R-RESCUE-reflowoven
- C10, C11, C12, C7, C8, C9: symbol C -> C-RESCUE-reflowoven
- R10, R7, R8, R9: symbol R -> R-RESCUE-reflowoven
Connections:
- wire segments 76 -> 87
