File: hardware/reflowoven.kicad_sch (KiCad schematic)
At the start: 23 parts, among them P1 USB-A-SHLD, P2 CONN_6, P3 CONN_2, P4 CONN_2, P5 CONN_01X08, U1 MSP430G2553IPW20, U2 FT232RL, U3 LM317, X1 CRYSTAL

Commit message: Updated schematic and PCB to 100% match footprints
Parts:
- C1: footprint Capacitors_SMD:C_0603 -> Capacitor_SMD:C_0603_1608Metric
Changed lines of the file:
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@@
       (effects (font (size 1.27 1.27)) (justify left))
     )
-    (property "Footprint" "Capacitors_SMD:C_0603" (id 2) (at 74.93 30.7848 0)
+    (property "Footprint" "Capacitor_SMD:C_0603_1608Metric" (id 2) (at 74.93 30.7848 0)
       (effects (font (size 1.27 1.27)) hide)
     )
@@
     )
     (path "/32dae22d-3d38-4916-a6c3-5108b29835c8"
-      (reference "C1") (unit 1) (value "100nF") (footprint "Capacitors_SMD:C_0603")
+      (reference "C1") (unit 1) (value "100nF") (footprint "Capacitor_SMD:C_0603_1608Metric")
     )
     (path "/00000000-0000-0000-0000-000050fb8dfc"
@@
       (reference "U3") (unit 1) (value "LM317") (footprint "Package_TO_SOT_THT:TO-220-3_Vertical")
     )
+    (path "/00000000-0000-0000-0000-000058bc1d4b/06e8525a-7bab-4869-ac74-e17ab11d8f41"
+      (reference "U4") (unit 1) (value "ULN2003A") (footprint "Package_SO:SO-16_3.9x9.9mm_P1.27mm")
+    )
     (path "/00000000-0000-0000-0000-000058bc1d4b/00000000-0000-0000-0000-000058bc28ba"
       (reference "U5") (unit 1) (value "MCHRM3H") (footprint "svolpe-custom-mod:MCHRM3H")
@@
       (reference "U8") (unit 1) (value "MCHRM3H") (footprint "svolpe-custom-mod:MCHRM3H")
     )
-    (path "/00000000-0000-0000-0000-000058bc1d4b/06e8525a-7bab-4869-ac74-e17ab11d8f41"
-      (reference "U?") (unit 1) (value "ULN2003A") (footprint "Housings_SOIC:SOIC-16_3.9x9.9mm_Pitch1.27mm")
-    )
     (path "/00000000-0000-0000-0000-000050fb9344"
